File: hardware/load-cell.kicad_pcb (KiCad board)
At the start: 2 copper layers, 30 x 30 mm, 36 parts, among them P1 CON-SENSOR, P2 Boot, P3 Debug, P4 AKL_5_2, P5 AKL_5_2, U1 XMC1XXX24, U2 FAN4860, U3 HX711, U4 DRILL, U5 DRILL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

Commit message: change "Status" and "LED" led colors
Parts:
- D1: value blue -> green
- D2: value green -> blue
Changed lines of the file:
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@@
       (effects (font (size 0.2 0.2) (thickness 0.05)))
     )
-    (fp_text value green (at 0.75 0.45 180) (layer F.Fab)
+    (fp_text value blue (at 0.75 0.45 180) (layer F.Fab)
       (effects (font (size 0.2 0.2) (thickness 0.05)))
     )
@@
       (effects (font (size 0.2 0.2) (thickness 0.05)))
     )
-    (fp_text value blue (at 0.75 0.45) (layer F.Fab)
-      (effects (font (size 0.2 0.2) (thickness 0.05)))
-    )
+    (fp_text value green (at 0.75 0.45) (layer F.Fab)
+      (effects (font (size 0.2 0.2) (thickness 0.05)))
+    )
